File: PhoneSwitchPCBs/PhoneInterface/PhoneInterface.kicad_pcb (KiCad board)
At the start: 2 copper layers, 101.6 x 50.8 mm, 55 parts, among them J1 Interface, J2 6P2C, K1 EC2-5NU, K2 EC2-5NU, K4 EC2-5NU, K5 EC2-5NU, Q1 PHPT61003PYX, Q2 PHPT61003NYX, Q3 XP231N02013R-G, Q4 XP231N02013R-G, Q5 XP231N02013R-G, Q6 XP231N02013R-G, U1 TCMD1000, U2 NL17SZ14DBVT1G

Commit message: Adapted and updated schematics and PCB design.
Converted schematics and board layouts to new file, as well as move design from one backplane to multiple modules.
Other:
- net class Default removed
