File: PhoneSwitchPCBs/ToneEncoderDecoder/ToneEncoderDecoder.kicad_pcb (KiCad board)
At the start: 2 copper layers, 93 x 70 mm, 124 parts, among them IC1 XRA1203IG24TR-F, IC2 NXB0108PWJ, IC3 74HC4316, IC4 74HC4316, IC5 TL074*DT, IC6 TL074*DT, IC7 TL072, IC8 MT8870DN1, IC9 MT8870DN1, J1 Tone Bus, J2 Power + Control, Q1 XP231N02013R-G, Q2 XP231N02013R-G, Y1 3.579545 MHz

Commit message: Added JLC text for number placement
Other:
- board text added: "JLCJLCJLCJLC"
Changed lines of the file:
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@@
   )
   (gr_rect (start 24.5 17.5) (end 117.5 87.5) (layer "Edge.Cuts") (width 0.1) (fill none))
+  (gr_text "JLCJLCJLCJLC" (at 26.2 50.9 90) (layer "B.SilkS")
+    (effects (font (size 1 1) (thickness 0.15)) (justify mirror))
+  )
   (gr_text "TeleTech MiniSwitch\nDTMF Decoder and Call Progress Tone Generator" (at 60.9 83.9) (layer "F.SilkS")
     (effects (font (size 1.5 1.5) (thickness 0.3)))
